Commit message: add contact sensors to main wheels

File: kobuki_description/urdf/kobuki_gazebo.urdf.xacro (robot description, xacro)
@@ -9,4 +9,11 @@
       <minDepth>0.001</minDepth>
       <maxVel>1.0</maxVel>
+      <sensor type="contact" name="wheel_left">
+        <always_on>1</always_on>
+        <update_rate>50.0</update_rate>
+        <visualize>true</visualize>
+        <contact>
+          <collision>wheel_left_link_collision</collision>
+        </contact>
     </gazebo>
     <gazebo reference="wheel_right_link">
@@ -17,4 +24,11 @@
       <minDepth>0.001</minDepth>
       <maxVel>1.0</maxVel>
+      <sensor type="contact" name="wheel_right">
+        <always_on>1</always_on>
+        <update_rate>50.0</update_rate>
+        <visualize>true</visualize>
+        <contact>
+          <collision>wheel_right_link_collision</collision>
+        </contact>
     </gazebo>
     <gazebo reference="caster_front_link">
@@ -175,4 +189,6 @@
         <bumper_name>bumpers</bumper_name>
         <imu_name>imu</imu_name>
+        <wheel_left_sensor_name>wheel_left</wheel_left_sensor_name>
+        <wheel_right_sensor_name>wheel_right</wheel_right_sensor_name>
       </plugin>
     </gazebo>

Commit message: add contact sensors to caster wheels

File: kobuki_description/urdf/kobuki_gazebo.urdf.xacro (robot description, xacro)
@@ -39,4 +39,11 @@
       <minDepth>0.001</minDepth>
       <maxVel>1.0</maxVel>
+      <sensor type="contact" name="caster_front">
+        <always_on>1</always_on>
+        <update_rate>50.0</update_rate>
+        <visualize>true</visualize>
+        <contact>
+          <collision>base_footprint_fixed_joint_lump__caster_front_link_collision_2</collision>
+        </contact>
     </gazebo>
     <gazebo reference="caster_back_link">
@@ -47,4 +54,11 @@
       <minDepth>0.001</minDepth>
       <maxVel>1.0</maxVel>
+      <sensor type="contact" name="caster_back">
+        <always_on>1</always_on>
+        <update_rate>50.0</update_rate>
+        <visualize>true</visualize>
+        <contact>
+          <collision>base_footprint_fixed_joint_lump__caster_back_link_collision_1</collision>
+        </contact>
     </gazebo>
     <gazebo reference="base_link">
@@ -191,4 +205,6 @@
         <wheel_left_sensor_name>wheel_left</wheel_left_sensor_name>
         <wheel_right_sensor_name>wheel_right</wheel_right_sensor_name>
+        <caster_front_sensor_name>caster_front</caster_front_sensor_name>
+        <caster_back_sensor_name>caster_back</caster_back_sensor_name>
       </plugin>
     </gazebo>
